Commit message: Removing unecessary stuff

File: robot_bringup/urdf/gazebo_control.xacro (robot description, xacro)
@@ -4,5 +4,4 @@
       <plugin filename="gz-sim-joint-state-publisher-system" name="gz::sim::systems::JointStatePublisher">
          <topic>joint_states</topic>
-         <!-- <joint_name>cg_joint</joint_name>s -->
          <joint_name>rr_wheel_joint</joint_name>
          <joint_name>rl_wheel_joint</joint_name>

File: robot_bringup/urdf/robot.urdf.xacro (robot description, xacro)
@@ -3,4 +3,3 @@
     <xacro:include filename="robot_core.xacro" />
     <xacro:include filename="gazebo_control.xacro" />
-    <!-- <xacro:include filename="lidar.xacro" /> -->
 </robot>

File: robot_bringup/urdf/robot_core.xacro (robot description, xacro)
@@ -63,40 +63,10 @@
       </xacro:inertial_box>
    </link>
-   <!-- <joint name="cg_joint" type="continuous">
-      <parent link="base_link"/>
-      <child link="cg_link"/>
-      <origin xyz="0.0 ${base_width/2 + wheel_width/2} ${wheel_zoff}" rpy="${-pi/2} 0.0 0.0"/>
-      <axis xyz="0 0 1"/>
-   </joint>
-   <link name="cg_link">
-      <visual>
-            <geometry>
-               <cylinder radius="${wheel_radius}" length="${wheel_width}"/>
-            </geometry>
-            <material name = "Green">
-               <color rgba= "0.0 1.0 0.0 1"/>
-            </material>
-      </visual>
-      <collision>
-            <geometry>
-               <cylinder radius="${wheel_radius}" length="${wheel_width}"/>
-            </geometry>
-      </collision>
-      <xacro:inertial_cylinder mass="${wheel_mass}"  radius="${wheel_radius}" length="${wheel_width}">
-            <origin xyz="0 0 0" rpy="0 0 0"/>
-      </xacro:inertial_cylinder>
-   </link> -->
    <xacro:create_wheel prefix="rl_wheel" x_reflect="-1" y_reflect="1" x="${wheel_xoff}" y="${wheel_yoff}" z="${wheel_zoff}" b="${base_width}" r="${wheel_radius}" w="${wheel_width}" m="${wheel_mass}" />
    <xacro:create_wheel prefix="rr_wheel" x_reflect="-1" y_reflect="-1" x="${wheel_xoff}" y="${wheel_yoff}" z="${wheel_zoff}" b="${base_width}" r="${wheel_radius}" w="${wheel_width}" m="${wheel_mass}" />
    <xacro:create_wheel prefix="fl_wheel" x_reflect="1" y_reflect="1" x="${wheel_xoff}" y="${wheel_yoff}" z="${wheel_zoff}" b="${base_width}" r="${wheel_radius}" w="${wheel_width}" m="${wheel_mass}" />
    <xacro:create_wheel prefix="fr_wheel" x_reflect="1" y_reflect="-1" x="${wheel_xoff}" y="${wheel_yoff}" z="${wheel_zoff}" b="${base_width}" r="${wheel_radius}" w="${wheel_width}" m="${wheel_mass}" />
-   <!-- <xacro:create_wheel prefix="cg" x_reflect="0" y_reflect="-0.5" x="${wheel_xoff}" y="${wheel_yoff}" z="${wheel_zoff}" b="${base_width}" r="${wheel_radius}" w="${wheel_width}" m="${wheel_mass}" /> -->
-   <!-- <xacro:create_wheel prefix="cg" x_reflect="0" y_reflect="0" x="0" y="-0.5" z="0" b="${base_width}" r="${wheel_radius}" w="${wheel_width}" m="${wheel_mass}" /> -->
    <gazebo reference="base_link"/>
    <gazebo reference="cart_link"/>
-   <gazebo reference="cg_link">
-      <mu1>1.0</mu1>
-      <mu2>1.0</mu2>
-   </gazebo>
    <gazebo reference="rl_wheel_link">
       <mu1>1.0</mu1>
